Commit message: adds super awesome scan

File: common/test/urdf/r2d2_robot/r2d2_bottom_heavy.urdf (robot description, URDF)
Before this commit: robot r2d2, 13 links, 12 joints
Joints:
- joint base_link_to_laser_body: origin xyz=0.25 0.0 -0.4 rpy=0 0 0 -> xyz=0.25 0.0 -0.45 rpy=0 0 0

File: common/test/urdf/r2d2_robot/r2d2_bottom_heavy.urdf.xacro (robot description, xacro)
@@ -30,5 +30,5 @@
     <parent link="base_link"/>
     <child link="${laser_name}_laser_body"/>
-    <origin xyz="0.25 0.0 -0.4" rpy="0 0 0" />
+    <origin xyz="0.25 0.0 -0.45" rpy="0 0 0" />
   </joint>
   <link name="right_leg">
